File: esp-printer.sch (KiCad schematic (older format))
At the start: 65 parts, among them CON1 BARREL_JACK, P1 USB_OTG, P2 CONN_01X02, P3 CONN_01X06, P4 CONN_01X06, P5 CONN_01X08, P6 CONN_01X08, Q1 Q_NMOS_GSD, Q2 Q_NMOS_GSD, SW1 SW_PUSH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

Commit message: Assign footprints with cvpcb
Parts:
- C1, C5: footprint (none) -> Capacitors_SMD:C_0805_HandSoldering
- C10, C11, C12, C13, C14, C2, C3, C4, C6, C7, C8, C9: footprint (none) -> Capacitors_SMD:C_0603_HandSoldering
- CON1: footprint (none) -> guri-lib:MJ-179PH
- D1, D2, D4, D6, D7, D8, D9: footprint (none) -> LEDs:LED-0603
- D3, D5: footprint (none) -> Diodes_SMD:SOD-123
- L1: footprint (none) -> Resistors_SMD:R_0805_HandSoldering
- P1: footprint (none) -> Connect:USB_Micro-B
- P2: footprint (none) -> guri-lib:B2P-VH
- P3, P4: footprint (none) -> Socket_Strips:Socket_Strip_Straight_1x06
- P5, P6: footprint (none) -> Socket_Strips:Socket_Strip_Straight_1x08
- Q1, Q2: footprint (none) -> TO_SOT_Packages_SMD:SOT-23_Handsoldering
- R1, R10, R11, R12, R13, R14, R15, R16, R17, R18, R19, R2, R3, R4, R5, R6, R7, R8, R9: footprint (none) -> Resistors_SMD:R_0603_HandSoldering
- SW1, SW2: footprint (none) -> guri-lib:SKRPACE010
- TS1, TS2, TS3, TS4: footprint (none) -> guri-lib:TouchPad_Arrow
- TS5, TS6, TS7: footprint (none) -> guri-lib:TouchPad_Square
- U1: footprint (none) -> SMD_Packages:SOIC-8-N
- U2: footprint (none) -> guri-lib:AQM1602XA
- U3: footprint (none) -> guri-lib:ESP-WROOM-32
- U4: footprint (none) -> SMD_Packages:SSOP-20

Commit message: Add a PCB pattern
Parts:
- removed P3, P4: CONN_01X06, Socket_Strips:Socket_Strip_Straight_1x06, symbol CONN_01X06
- removed P5, P6: CONN_01X08, Socket_Strips:Socket_Strip_Straight_1x08, symbol CONN_01X08
- added U5: ArduinoUno-R1, guri-lib:ArduinoUno-R1, symbol ArduinoUno-R1
- D8: value LED -> WIFI
- D9: value LED -> STATUS
- P1: footprint Connect:USB_Micro-B -> guri-lib:ZX62R-B-5P
Connections:
- net GND: now also U5.15 (GND), U5.24 (GND), U5.25 (GND)
- net PRINTER_+5V: now also U5.26 (5V)
- net PRINTER_DATA: now also U5.2 (D1/TX)
Other:
- moved on the sheet: P2
Changed lines of the file:
@@
 EESchema Schematic File Version 2
+LIBS:guri-lib
 LIBS:power
 LIBS:device
@@
 LIBS:contrib
 LIBS:valves
-LIBS:guri-lib
 LIBS:esp-printer-cache
 EELAYER 25 0
@@
 F 0 "P1" H 5425 1675 50  0000 C CNN
 F 1 "USB_OTG" H 5100 2000 50  0000 C CNN
-F 2 "Connect:USB_Micro-B" V 5050 1700 50  0001 C CNN
+F 2 "guri-lib:ZX62R-B-5P" V 5050 1700 50  0001 C CNN
 F 3 "" V 5050 1700 50  0000 C CNN
 	1    5100 1800
@@
 Wire Wire Line
 	5500 5850 5500 5900
-$Comp
-L CONN_01X08 P6
-U 1 1 59941E93
-P 10100 3750
-F 0 "P6" H 10100 4200 50  0000 C CNN
-F 1 "CONN_01X08" V 10200 3750 50  0000 C CNN
-F 2 "Socket_Strips:Socket_Strip_Straight_1x08" H 10100 3750 50  0001 C CNN
-F 3 "" H 10100 3750 50  0000 C CNN
-	1    10100 3750
-	-1   0    0    1
-$EndComp
-$Comp
-L CONN_01X08 P5
-U 1 1 59941F69
-P 10100 2850
-F 0 "P5" H 10100 3300 50  0000 C CNN
-F 1 "CONN_01X08" V 10200 2850 50  0000 C CNN
-F 2 "Socket_Strips:Socket_Strip_Straight_1x08" H 10100 2850 50  0001 C CNN
-F 3 "" H 10100 2850 50  0000 C CNN
-	1    10100 2850
-	-1   0    0    1
-$EndComp
-$Comp
-L CONN_01X06 P4
-U 1 1 59942036
-P 9800 3850
-F 0 "P4" H 9800 4200 50  0000 C CNN
-F 1 "CONN_01X06" V 9900 3850 50  0000 C CNN
-F 2 "Socket_Strips:Socket_Strip_Straight_1x06" H 9800 3850 50  0001 C CNN
-F 3 "" H 9800 3850 50  0000 C CNN
-	1    9800 3850
-	1    0    0    -1
-$EndComp
-$Comp
-L CONN_01X06 P3
-U 1 1 599420FF
-P 9800 2950
-F 0 "P3" H 9800 3300 50  0000 C CNN
-F 1 "CONN_01X06" V 9900 2950 50  0000 C CNN
-F 2 "Socket_Strips:Socket_Strip_Straight_1x06" H 9800 2950 50  0001 C CNN
-F 3 "" H 9800 2950 50  0000 C CNN
-	1    9800 2950
-	1    0    0    -1
-$EndComp
-NoConn ~ 10300 3200
-NoConn ~ 10300 3100
-NoConn ~ 10300 3000
-NoConn ~ 10300 2900
-NoConn ~ 10300 2800
-NoConn ~ 10300 2700
-NoConn ~ 10300 2500
-NoConn ~ 9600 4100
-NoConn ~ 9600 4000
-NoConn ~ 9600 3900
-NoConn ~ 9600 3800
-NoConn ~ 9600 3700
-NoConn ~ 9600 3600
-NoConn ~ 9600 3200
-NoConn ~ 9600 2700
-NoConn ~ 9600 2800
+NoConn ~ 10400 3200
+NoConn ~ 10400 3100
+NoConn ~ 10400 3000
+NoConn ~ 10400 2900
+NoConn ~ 10400 2800
+NoConn ~ 10400 2700
+NoConn ~ 10400 2500
+NoConn ~ 9400 4100
+NoConn ~ 9400 4000
+NoConn ~ 9400 3900
+NoConn ~ 9400 3800
+NoConn ~ 9400 3700
+NoConn ~ 9400 3600
+NoConn ~ 9400 3400
+NoConn ~ 9400 2900
+NoConn ~ 9400 3000
 Wire Wire Line
 	2500 900  2500 1200
@@
 Text GLabel 2600 1200 2    60   Output ~ 0
 PRINTER_+5V
-Text GLabel 9500 2900 0    60   Input ~ 0
+Text GLabel 9300 3100 0    60   Input ~ 0
 PRINTER_+5V
 Wire Wire Line
-	9600 2900 9500 2900
+	9400 3100 9300 3100
 $Comp
 L GND #PWR043
 U 1 1 59943664
-P 9450 3150
-F 0 "#PWR043" H 9450 2900 50  0001 C CNN
-F 1 "GND" H 9450 3000 50  0000 C CNN
-F 2 "" H 9450 3150 50  0000 C CNN
-F 3 "" H 9450 3150 50  0000 C CNN
-	1    9450 3150
-	1    0    0    -1
-$EndComp
-Wire Wire Line
-	9600 3000 9450 3000
-Wire Wire Line
-	9450 3000 9450 3150
-Wire Wire Line
-	9600 3100 9450 3100
-Connection ~ 9450 3100
+P 9250 3350
+F 0 "#PWR043" H 9250 3100 50  0001 C CNN
+F 1 "GND" H 9250 3200 50  0000 C CNN
+F 2 "" H 9250 3350 50  0000 C CNN
+F 3 "" H 9250 3350 50  0000 C CNN
+	1    9250 3350
+	1    0    0    -1
+$EndComp
+Wire Wire Line
+	9400 3200 9250 3200
+Wire Wire Line
+	9250 3200 9250 3350
+Wire Wire Line
+	9400 3300 9250 3300
+Connection ~ 9250 3300
 $Comp
 L GND #PWR044
 U 1 1 5994393F
-P 10450 2700
-F 0 "#PWR044" H 10450 2450 50  0001 C CNN
-F 1 "GND" H 10450 2550 50  0000 C CNN
-F 2 "" H 10450 2700 50  0000 C CNN
-F 3 "" H 10450 2700 50  0000 C CNN
-	1    10450 2700
-	1    0    0    -1
-$EndComp
-Wire Wire Line
-	10450 2700 10450 2600
-Wire Wire Line
-	10450 2600 10300 2600
-NoConn ~ 10300 4100
-NoConn ~ 10300 3900
-NoConn ~ 10300 3800
-NoConn ~ 10300 3700
-NoConn ~ 10300 3600
-NoConn ~ 10300 3500
-Wire Wire Line
-	10300 4000 10400 4000
-Text GLabel 10400 4000 2    60   Input ~ 0
+P 10550 2700
+F 0 "#PWR044" H 10550 2450 50  0001 C CNN
+F 1 "GND" H 10550 2550 50  0000 C CNN
+F 2 "" H 10550 2700 50  0000 C CNN
+F 3 "" H 10550 2700 50  0000 C CNN
+	1    10550 2700
+	1    0    0    -1
+$EndComp
+Wire Wire Line
+	10550 2700 10550 2600
+Wire Wire Line
+	10550 2600 10400 2600
+NoConn ~ 10400 4100
+NoConn ~ 10400 3900
+NoConn ~ 10400 3800
+NoConn ~ 10400 3700
+NoConn ~ 10400 3600
+NoConn ~ 10400 3500
+Wire Wire Line
+	10400 4000 10500 4000
+Text GLabel 10500 4000 2    60   Input ~ 0
 PRINTER_DATA
-NoConn ~ 10300 3400
+NoConn ~ 10400 3400
 $Comp
 L CONN_01X02 P2
 U 1 1 59944DD2
-P 9350 3900
-F 0 "P2" H 9350 4050 50  0000 C CNN
-F 1 "CONN_01X02" V 9450 3900 50  0000 C CNN
-F 2 "guri-lib:B2P-VH" H 9350 3900 50  0001 C CNN
-F 3 "" H 9350 3900 50  0000 C CNN
-	1    9350 3900
+P 9050 4150
+F 0 "P2" H 9050 4300 50  0000 C CNN
+F 1 "CONN_01X02" V 9150 4150 50  0000 C CNN
+F 2 "guri-lib:B2P-VH" H 9050 4150 50  0001 C CNN
+F 3 "" H 9050 4150 50  0000 C CNN
+	1    9050 4150
 	1    0    0    -1
 $EndComp
@@
 L GND #PWR045
 U 1 1 59944F9E
-P 9050 4050
-F 0 "#PWR045" H 9050 3800 50  0001 C CNN
-F 1 "GND" H 9050 3900 50  0000 C CNN
-F 2 "" H 9050 4050 50  0000 C CNN
-F 3 "" H 9050 4050 50  0000 C CNN
-	1    9050 4050
-	1    0    0    -1
-$EndComp
-Wire Wire Line
-	9150 3950 9050 3950
-Wire Wire Line
-	9050 3950 9050 4050
-Wire Wire Line
-	9150 3850 9050 3850
-Wire Wire Line
-	9050 3850 9050 3750
-Text GLabel 9050 3750 1    60   Input ~ 0
+P 8750 4300
+F 0 "#PWR045" H 8750 4050 50  0001 C CNN
+F 1 "GND" H 8750 4150 50  0000 C CNN
+F 2 "" H 8750 4300 50  0000 C CNN
+F 3 "" H 8750 4300 50  0000 C CNN
+	1    8750 4300
+	1    0    0    -1
+$EndComp
+Wire Wire Line
+	8850 4200 8750 4200
+Wire Wire Line
+	8750 4200 8750 4300
+Wire Wire Line
+	8850 4100 8750 4100
+Wire Wire Line
+	8750 4100 8750 4000
+Text GLabel 8750 4000 1    60   Input ~ 0
 PRINTER_+5V
 Wire Wire Line
@@
 P 10100 5650
 F 0 "D8" H 10100 5750 50  0000 C CNN
-F 1 "LED" H 10100 5550 50  0000 C CNN
+F 1 "WIFI" H 10100 5550 50  0000 C CNN
 F 2 "LEDs:LED-0603" H 10100 5650 50  0001 C CNN
 F 3 "" H 10100 5650 50  0000 C CNN
@@
 P 10400 5650
 F 0 "D9" H 10400 5750 50  0000 C CNN
-F 1 "LED" H 10400 5550 50  0000 C CNN
+F 1 "STATUS" H 10400 5550 50  0000 C CNN
 F 2 "LEDs:LED-0603" H 10400 5650 50  0001 C CNN
 F 3 "" H 10400 5650 50  0000 C CNN
@@
 NoConn ~ 7000 4300
 NoConn ~ 5100 4900
+$Comp
+L ArduinoUno-R1 U5
+U 1 1 59B9D25A
+P 9900 3300
+F 0 "U5" H 9900 4250 60  0000 C CNN
+F 1 "ArduinoUno-R1" H 9900 2350 60  0000 C CNN
+F 2 "guri-lib:ArduinoUno-R1" H 9900 3300 60  0001 C CNN
+F 3 "" H 9900 3300 60  0000 C CNN
+	1    9900 3300
+	1    0    0    -1
+$EndComp
 $EndSCHEMATC
