File: esp-printer.kicad_pcb (KiCad board)
At the start: 2 copper layers, 110 x 170 mm, 70 parts, among them CON1 BARREL_JACK, P1 USB_OTG, P2 CONN_01X02, Q1 Q_NMOS_GSD, Q2 Q_NMOS_GSD, SW1 SW_PUSH, SW2 SW_PUSH, U1 LT1963A, U2 AQM1602XA, U3 ESP-WROOM-32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

Commit message: Output gerber files for manufacturing
Parts:
- moved P2 9.00 mm to (116.5, 74.0)
Routing:
- net PRINTER_+5V: track 124.7 -> 119.7 mm
- net GND: track 604.3 -> 599.5 mm, vias 8 -> 9
- net +3V3: track 254.9 -> 254.1 mm
Other:
- board text added: "ISP"
- board text added: "RESET"
